Commit message: Uncompleted changes for visual and box size. Model able to load in gazebo

File: models/soccerbot v4/model.urdf (robot description, URDF)
Before this commit: robot soccerbot_noarms, 22 links, 21 joints
Links:
- link left_foot: geometry collision box size=0.09 0.03674 0.07; visual mesh filename=package://soccer_description/meshes/soccerbot v4/Left Foot.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 scale=0.001 0.001 0.001
