Commit message: Updated Materials

File: models/soccerbot/model.xacro (robot description, xacro)
@@ -1,10 +1,8 @@
 <?xml version="1.0" ?>
-<robot name="soccerbot_noarms">
-    <gazebo>
-        <plugin name="gazebo_ros_control" filename="libgazebo_ros_control.so">
-            <robotNamespace>/soccerbot</robotNamespace>
-            <robotSimType>gazebo_ros_control/DefaultRobotHWSim</robotSimType>
-        </plugin>
-    </gazebo>
+<robot name="soccerbot" xmlns:xacro="http://www.ros.org/wiki/xacro">
+    <xacro:property name="PI" value="3.1415926535897931"/>
+    <xacro:include filename="$(find soccer_description)/models/soccerbot/model.gazebo" />
+    <!-- Import Rviz colors -->
+    <xacro:include filename="$(find soccer_description)/models/soccerbot/materials.xacro" />
     <!-- Joint to keep the robot up in midair -->
     <!--   <link name="world" />
@@ -16,5 +14,5 @@
       </joint> -->
     <!-- Links -->
-    <link name="base_link"/>
+    <link name="base_link" />
     <link name="torso">
         <inertial>
@@ -36,63 +34,6 @@
         </visual>
     </link>
-    <link name="camera"/>
-    <gazebo reference="camera">
-        <sensor name='main_camera' type='camera'>
-            <update_rate>10</update_rate>
-            <camera name='__default__'>
-                <horizontal_fov>1.39626</horizontal_fov>
-                <image>
-                    <width>640</width>
-                    <height>480</height>
-                    <format>R8G8B8</format>
-                </image>
-                <clip>
-                    <near>1</near>
-                    <far>100</far>
-                </clip>
-                <noise>
-                    <type>gaussian</type>
-                    <mean>0</mean>
-                    <stddev>0.007</stddev>
-                </noise>
-            </camera>
-            <always_on>1</always_on>
-            <visualize>1</visualize>
-            <plugin name='camera_controller' filename='libgazebo_ros_camera.so'>
-                <alwaysOn>true</alwaysOn>
-                <updateRate>0.0</updateRate>
-                <cameraName>soccerbot/camera1</cameraName>
-                <imageTopicName>image_raw</imageTopicName>
-                <cameraInfoTopicName>camera_info</cameraInfoTopicName>
-                <frameName>camera_link</frameName>
-                <hackBaseline>0.07</hackBaseline>
-                <distortionK1>0.0</distortionK1>
-                <distortionK2>0.0</distortionK2>
-                <distortionK3>0.0</distortionK3>
-                <distortionT1>0.0</distortionT1>
-                <distortionT2>0.0</distortionT2>
-            </plugin>
-        </sensor>
-    </gazebo>
-    <link name="imu"/>
-    <gazebo reference="imu">
-        <gravity>true</gravity>
-        <sensor name="imu_sensor" type="imu">
-            <always_on>true</always_on>
-            <update_rate>100</update_rate>
-            <visualize>true</visualize>
-            <topic>__default_topic__</topic>
-            <plugin filename="libgazebo_ros_imu_sensor.so" name="imu_plugin">
-                <topicName>soccerbot/imu</topicName>
-                <bodyName>imu_link</bodyName>
-                <updateRateHZ>50.0</updateRateHZ>
-                <gaussianNoise>0.0</gaussianNoise>
-                <xyzOffset>0 0 0</xyzOffset>
-                <rpyOffset>0 0 0</rpyOffset>
-                <frameName>imu_link</frameName>
-            </plugin>
-            <pose>0 0 0 0 0 0</pose>
-        </sensor>
-    </gazebo>
+    <link name="camera" />
+    <link name="imu" />
     <link name="head">
         <inertial>
@@ -112,4 +53,5 @@
                 <mesh filename="package://soccer_description/meshes/soccerbot v4/Head.stl" scale="0.001 0.001 0.001"/>
             </geometry>
+            <material name="black" />
         </visual>
     </link>
@@ -129,7 +71,7 @@
             <origin rpy="0  0  0" xyz="0  0  0"/>
             <geometry>
-                <mesh filename="package://soccer_description/meshes/soccerbot v4/Left Ankle.stl"
-                      scale="0.001 0.001 0.001"/>
-            </geometry>
+                <mesh filename="package://soccer_description/meshes/soccerbot v4/Left Ankle.stl" scale="0.001 0.001 0.001"/>
+            </geometry>
+            <material name="black" />
         </visual>
     </link>
@@ -149,7 +91,7 @@
             <origin rpy="0  0  0" xyz="0 -0.0827  0"/>
             <geometry>
-                <mesh filename="package://soccer_description/meshes/soccerbot v4/Left Calve.stl"
-                      scale="0.001 0.001 0.001"/>
-            </geometry>
+                <mesh filename="package://soccer_description/meshes/soccerbot v4/Left Calve.stl" scale="0.001 0.001 0.001"/>
+            </geometry>
+            <material name="black" />
         </visual>
     </link>
@@ -160,123 +102,17 @@
             <inertia ixx="0.026" ixy="0" ixz="0" iyy="0.023" iyz="0" izz="0.013"/>
         </inertial>
-        <collision name="pressure_pad_1">
-            <pose>0.45 0.45 -0.1 0 43.5 4.5</pose>
-            <geometry>
-                <box size="0.1 0.1 0.02" />
-            </geometry>
-            <surface>
-                <contact>
-                    <ode>
-                        <kp>100000</kp>
-                        <kd>1</kd>
-                    </ode>
-                </contact>
-                <friction>
-                    <ode>
-                        <mu>1</mu>
-                        <mu2>1</mu2>
-                    </ode>
-                </friction>
-            </surface>
-        </collision>
-        <collision name="pressure_pad_2">
-            <pose>0.45 -0.45 -0.1 0 -16.5 4.5</pose>
-            <geometry>
-                <box size="0.1 0.1 0.02" />
-            </geometry>
-            <surface>
-                <contact>
-                    <ode>
-                        <kp>100000</kp>
-                        <kd>1</kd>
-                    </ode>
-                </contact>
-                <friction>
-                    <ode>
-                        <mu>1</mu>
-                        <mu2>1</mu2>
-                    </ode>
-                </friction>
-            </surface>
-        </collision>
-        <collision name="pressure_pad_3">
-            <pose>-0.45 0.45 -0.1 0 -16.5 -75.5</pose>
-            <geometry>
-                <box size = "0.05 0.05 0.02" />
-            </geometry>
-            <surface>
-                <contact>
-                    <ode>
-                        <kp>100000</kp>
-                        <kd>1</kd>
-                    </ode>
-                </contact>
-                <friction>
-                    <ode>
-                        <mu>1</mu>
-                        <mu2>1</mu2>
-                    </ode>
-                </friction>
-            </surface>
-        </collision>
-        <collision name="pressure_pad_4">
-            <pose>-0.45 -0.45 -0.1 0 43.5 -75.5</pose>
-            <geometry>
-                <box size="0.05 0.05 0.02" />
-            </geometry>
-            <surface>
-                <contact>
-                    <ode>
-                        <kp>100000</kp>
-                        <kd>1</kd>
-                    </ode>
-                </contact>
-                <friction>
-                    <ode>
-                        <mu>1</mu>
-                        <mu2>1</mu2>
-                    </ode>
-                </friction>
-            </surface>
-        </collision>
-        <visual name="pressure_pad_1">
-            <pose>0.45 0.45 -0.1 0 43.5 4.5</pose>
-            <geometry>
-                <box size="0.1 0.1 0.02" />
-            </geometry>
-        </visual>
-        <visual name="pressure_pad_2">
-            <pose>0.45 -0.45 -0.1 0 -16.5 4.5</pose>
-            <geometry>
-                <box size="0.1 0.1 0.02" />
-            </geometry>
-        </visual>
-        <visual name="pressure_pad_3">
-            <pose>-0.45 0.45 -0.1 0 -16.5 -75.5</pose>
-            <geometry>
-                <box size="0.05 0.05 0.02" />
-            </geometry>
-        </visual>
-        <visual name="pressure_pad_4">
-            <pose>-0.45 -0.45 -0.1 0 43.5 -75.5</pose>
-            <geometry>
-                <box size="0.05 0.05 0.02" />
-            </geometry>
-        </visual>
-        <sensor name="my_contact" type="contact">
-            <contact>
-                <collision>pressure_pad_1</collision>
-                <collision>pressure_pad_2</collision>
-                <collision>pressure_pad_3</collision>
-                <collision>pressure_pad_4</collision>
-            </contact>
-            <plugin name="my_plugin" filename="libPressurePlugin.so"/>
-        </sensor>
-        <visual name="visual">
-            <origin rpy="0  0  0" xyz="0  0  0"/>
-            <geometry>
-                <mesh filename="package://soccer_description/meshes/soccerbot v4/Left Foot.stl"
-                      scale="0.001 0.001 0.001"/>
-            </geometry>
+        <collision name="collision">
+            <origin rpy="0 1.5708 0" xyz="-0.00401 -0.00737  0.00385"/>
+            <geometry>
+                <box size="0.09 0.03674 0.07"/>
+            </geometry>
+            <contact_coefficients mu ="100.0" />
+        </collision>
+        <visual name="visual">
+            <origin rpy="0  0  0" xyz="0  0  0"/>
+            <geometry>
+                <mesh filename="package://soccer_description/meshes/soccerbot v4/Left Foot.stl" scale="0.001 0.001 0.001"/>
+            </geometry>
+            <material name="black" />
         </visual>
     </link>
@@ -296,7 +132,7 @@
             <origin rpy="0  0  0" xyz="0  0  0"/>
             <geometry>
-                <mesh filename="package://soccer_description/meshes/soccerbot v4/Left Hip Front.stl"
-                      scale="0.001 0.001 0.001"/>
-            </geometry>
+                <mesh filename="package://soccer_description/meshes/soccerbot v4/Left Hip Front.stl" scale="0.001 0.001 0.001"/>
+            </geometry>
+            <material name="black" />
         </visual>
     </link>
@@ -316,7 +152,7 @@
             <origin rpy="0  0  0" xyz="0  0  0"/>
             <geometry>
-                <mesh filename="package://soccer_description/meshes/soccerbot v4/Left Hip Side.stl"
-                      scale="0.001 0.001 0.001"/>
-            </geometry>
+                <mesh filename="package://soccer_description/meshes/soccerbot v4/Left Hip Side.stl" scale="0.001 0.001 0.001"/>
+            </geometry>
+            <material name="black" />
         </visual>
     </link>
@@ -336,7 +172,7 @@
             <origin rpy="0  0  0" xyz="0  0  0"/>
             <geometry>
-                <mesh filename="package://soccer_description/meshes/soccerbot v4/Left Thigh.stl"
-                      scale="0.001 0.001 0.001"/>
-            </geometry>
+                <mesh filename="package://soccer_description/meshes/soccerbot v4/Left Thigh.stl" scale="0.001 0.001 0.001"/>
+            </geometry>
+            <material name="black" />
         </visual>
     </link>
@@ -358,4 +194,5 @@
                 <mesh filename="package://soccer_description/meshes/soccerbot v4/Neck.stl" scale="0.001 0.001 0.001"/>
             </geometry>
+            <material name="black" />
         </visual>
     </link>
@@ -375,7 +212,7 @@
             <origin rpy="0  0  0" xyz="0  0  0"/>
             <geometry>
-                <mesh filename="package://soccer_description/meshes/soccerbot v4/Right Ankle.stl"
-                      scale="0.001 0.001 0.001"/>
-            </geometry>
+                <mesh filename="package://soccer_description/meshes/soccerbot v4/Right Ankle.stl" scale="0.001 0.001 0.001"/>
+            </geometry>
+            <material name="black" />
         </visual>
     </link>
@@ -395,7 +232,7 @@
             <origin rpy="0  0  0" xyz="0     -0.0827  0"/>
             <geometry>
-                <mesh filename="package://soccer_description/meshes/soccerbot v4/Right Calve.stl"
-                      scale="0.001 0.001 0.001"/>
-            </geometry>
+                <mesh filename="package://soccer_description/meshes/soccerbot v4/Right Calve.stl" scale="0.001 0.001 0.001"/>
+            </geometry>
+            <material name="black" />
         </visual>
     </link>
@@ -411,12 +248,12 @@
                 <box size="0.09 0.03674 0.07"/>
             </geometry>
-            <contact_coefficients mu="100.0"/>
-        </collision>
-        <visual name="visual">
-            <origin rpy="0  0  0" xyz="0  0  0"/>
-            <geometry>
-                <mesh filename="package://soccer_description/meshes/soccerbot v4/Right Foot.stl"
-                      scale="0.001 0.001 0.001"/>
-            </geometry>
+            <contact_coefficients mu ="100.0" />
+        </collision>
+        <visual name="visual">
+            <origin rpy="0  0  0" xyz="0  0  0"/>
+            <geometry>
+                <mesh filename="package://soccer_description/meshes/soccerbot v4/Right Foot.stl" scale="0.001 0.001 0.001"/>
+            </geometry>
+            <material name="black" />
         </visual>
     </link>
@@ -436,7 +273,7 @@
             <origin rpy="0  0  0" xyz="0  0  0"/>
             <geometry>
-                <mesh filename="package://soccer_description/meshes/soccerbot v4/Right Hip Front.stl"
-                      scale="0.001 0.001 0.001"/>
-            </geometry>
+                <mesh filename="package://soccer_description/meshes/soccerbot v4/Right Hip Front.stl" scale="0.001 0.001 0.001"/>
+            </geometry>
+            <material name="black" />
         </visual>
     </link>
@@ -456,7 +293,7 @@
             <origin rpy="0  0  0" xyz="0  0  0"/>
             <geometry>
-                <mesh filename="package://soccer_description/meshes/soccerbot v4/Right Hip Side.stl"
-                      scale="0.001 0.001 0.001"/>
-            </geometry>
+                <mesh filename="package://soccer_description/meshes/soccerbot v4/Right Hip Side.stl" scale="0.001 0.001 0.001"/>
+            </geometry>
+            <material name="black" />
         </visual>
     </link>
@@ -476,7 +313,7 @@
             <origin rpy="0  0  0" xyz="0  0  0"/>
             <geometry>
-                <mesh filename="package://soccer_description/meshes/soccerbot v4/Right Thigh.stl"
-                      scale="0.001 0.001 0.001"/>
-            </geometry>
+                <mesh filename="package://soccer_description/meshes/soccerbot v4/Right Thigh.stl" scale="0.001 0.001 0.001"/>
+            </geometry>
+            <material name="black" />
         </visual>
     </link>
@@ -496,7 +333,7 @@
             <origin rpy="0  0  0" xyz="0  0  0"/>
             <geometry>
-                <mesh filename="package://soccer_description/meshes/soccerbot v4/Right Bicep.stl"
-                      scale="0.001 0.001 0.001"/>
-            </geometry>
+                <mesh filename="package://soccer_description/meshes/soccerbot v4/Right Bicep.stl" scale="0.001 0.001 0.001"/>
+            </geometry>
+            <material name="black" />
         </visual>
     </link>
@@ -516,7 +353,7 @@
             <origin rpy="0  0  0" xyz="0  0  0"/>
             <geometry>
-                <mesh filename="package://soccer_description/meshes/soccerbot v4/Left Bicep.stl"
-                      scale="0.001 0.001 0.001"/>
-            </geometry>
+                <mesh filename="package://soccer_description/meshes/soccerbot v4/Left Bicep.stl" scale="0.001 0.001 0.001"/>
+            </geometry>
+            <material name="black" />
         </visual>
     </link>
@@ -536,7 +373,7 @@
             <origin rpy="0  0  0" xyz="0  0  0"/>
             <geometry>
-                <mesh filename="package://soccer_description/meshes/soccerbot v4/Left Forearm.stl"
-                      scale="0.001 0.001 0.001"/>
-            </geometry>
+                <mesh filename="package://soccer_description/meshes/soccerbot v4/Left Forearm.stl" scale="0.001 0.001 0.001"/>
+            </geometry>
+            <material name="black" />
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