Commit message: Fixed Joint Angles

File: models/soccerbot/model.xacro (robot description, xacro)
@@ -17,18 +17,18 @@
     <link name="torso">
         <inertial>
-            <mass value="1219.727"/>
-            <origin rpy="1.57 0 1.57" xyz="0 0 -0.052"/>
-            <inertia ixx="8.01" ixy="0.075" ixz="0.032" iyy="3.08" iyz="0.708" izz="8.75"/>
-        </inertial>
-        <collision name="collision">
-            <origin rpy="1.5708 0 1.5708" xyz="0 0 -0.052"/>
-            <geometry>
-                <box size="0.152 0.145 0.130"/>
-            </geometry>
-        </collision>
-        <visual name="visual">
-            <origin rpy="1.5708 0 1.5708" xyz="0 0 0"/>
-            <geometry>
-                <mesh filename="package://soccer_description/meshes/soccerbot v4/Torso.stl" scale="0.001 0.001 0.001"/>
+            <mass value="1529.201"/>
+            <origin rpy="0 0 0" xyz="0 0 0"/>
+            <inertia ixx="5.590" ixy="0.006" ixz="0.063" iyy="8.698" iyz="-0.056" izz="3.302"/>
+        </inertial>
+        <collision name="collision">
+            <origin rpy="0 0 0" xyz="0 0 -0.052"/>
+            <geometry>
+                <box size="0.130 0.145 0.152"/>
+            </geometry>
+        </collision>
+        <visual name="visual">
+            <origin rpy="0 0 0" xyz="0 0 0"/>
+            <geometry>
+                <mesh filename="package://soccer_description/meshes/soccerbot v4/Torso.dae" scale="1 1 1"/>
             </geometry>
         </visual>
@@ -36,74 +36,154 @@
     <link name="camera" />
     <link name="imu" />
+    <link name="neck">
+        <inertial>
+            <mass value="11.294"/>
+            <origin rpy="0  0  0" xyz="0  0  0"/>
+            <inertia ixx="0.006" ixy="0" ixz="0" iyy="0.002" iyz="0" izz="0.005"/>
+        </inertial>
+        <collision name="collision">
+            <origin rpy="0  0  0" xyz="0 0 0.0165"/>
+            <geometry>
+                <box size="0.022 0.0523 0.033"/>
+            </geometry>
+        </collision>
+        <visual name="visual">
+            <origin rpy="0  0  0" xyz="0  0  0"/>
+            <geometry>
+                <mesh filename="package://soccer_description/meshes/soccerbot v4/Neck.dae" scale="1 1 1"/>
+            </geometry>
+            <material name="black" />
+        </visual>
+    </link>
     <link name="head">
         <inertial>
             <mass value="282.919"/>
             <origin rpy="0  0  0" xyz="0  0  0"/>
-            <inertia ixx="0.400" ixy="0" ixz="0" iyy="0.170" iyz="0.015" izz="0.392"/>
-        </inertial>
-        <collision name="collision">
-            <origin rpy="0  0  0" xyz="0 0.02648  0"/>
-            <geometry>
-                <box size="0.094 0.0779 0.0712"/>
-            </geometry>
-        </collision>
-        <visual name="visual">
-            <origin rpy="0  0  0" xyz="0  0  0"/>
-            <geometry>
-                <mesh filename="package://soccer_description/meshes/soccerbot v4/Head.stl" scale="0.001 0.001 0.001"/>
-            </geometry>
-            <material name="black" />
-        </visual>
-    </link>
-    <link name="left_ankle">
+            <inertia ixx="0.392" ixy="-0.011" ixz="-0.229" iyy="0.550" iyz="-0.011" izz="0.320"/>
+        </inertial>
+        <collision name="collision">
+            <origin rpy="0  0  0" xyz="0 0 0.01995"/>
+            <geometry>
+                <box size="0.0712 0.094 0.0839"/>
+            </geometry>
+        </collision>
+        <visual name="visual">
+            <origin rpy="0  0  0" xyz="0  0  0"/>
+            <geometry>
+                <mesh filename="package://soccer_description/meshes/soccerbot v4/Head.dae" scale="1 1 1"/>
+            </geometry>
+            <material name="black" />
+        </visual>
+    </link>
+    <link name="right_hip_side">
+        <inertial>
+            <mass value="9.364"/>
+            <origin rpy="0  0  0" xyz="0  0  0"/>
+            <inertia ixx="0.004" ixy="0" ixz="0" iyy="0.007" iyz="0" izz="0.004"/>
+        </inertial>
+        <collision name="collision">
+            <origin rpy="0  0  0" xyz="0 0 0.00899"/>
+            <geometry>
+                <box size="0.0475 0.022 0.039"/>
+            </geometry>
+        </collision>
+        <visual name="visual">
+            <origin rpy="0  0  0" xyz="0  0  0"/>
+            <geometry>
+                <mesh filename="package://soccer_description/meshes/soccerbot v4/Right Hip Side.dae" scale="1 1 1"/>
+            </geometry>
+            <material name="black" />
+        </visual>
+    </link>
+    <link name="right_hip_front">
+        <inertial>
+            <mass value="153.186"/>
+            <origin rpy="0 0 0" xyz="0 0 0"/>
+            <inertia ixx="0.060" ixy="0.000" ixz="-0.038" iyy="0.205" iyz="0.000" izz="0.173"/>
+        </inertial>
+        <collision name="collision">
+            <origin rpy="0 0 0" xyz="-0.02187 0 -0.01332"/>
+            <geometry>
+                <box size="0.083747 0.04885 0.0506"/>
+            </geometry>
+        </collision>
+        <visual name="visual">
+            <origin rpy="0  0  0" xyz="0  0  0"/>
+            <geometry>
+                <mesh filename="package://soccer_description/meshes/soccerbot v4/Right Hip Front.dae" scale="1 1 1"/>
+            </geometry>
+            <material name="black" />
+        </visual>
+    </link>
+    <link name="right_thigh">
+        <inertial>
+            <mass value="21.438"/>
+            <origin rpy="0 0 0" xyz="0  0  0"/>
+            <inertia ixx="0.063" ixy="0" ixz="0.002" iyy="0.063" iyz="0" izz="0.011"/>
+        </inertial>
+        <collision name="collision">
+            <origin rpy="0 0 0" xyz="0 0 -0.0445"/>
+            <geometry>
+                <box size="0.022 0.048 0.111"/>
+            </geometry>
+        </collision>
+        <visual name="visual">
+            <origin rpy="0  0  0" xyz="0  0  0"/>
+            <geometry>
+                <mesh filename="package://soccer_description/meshes/soccerbot v4/Right Thigh.dae" scale="1 1 1"/>
+            </geometry>
+            <material name="black" />
+        </visual>
+    </link>
+    <link name="right_calve">
+        <inertial>
+            <mass value="86.547"/>
+            <origin rpy="0  0  0" xyz="0 0 0"/>
+            <inertia ixx="0.072" ixy="0" ixz="0" iyy="0.443" iyz="0.003" izz="0.019"/>
+        </inertial>
+        <collision name="collision">
+            <origin rpy="0 0 0" xyz="0 0 -0.03385"/>
+            <geometry>
+                <box size="0.031883 0.048 0.105683"/>
+            </geometry>
+        </collision>
+        <visual name="visual">
+            <origin rpy="0 0 0" xyz="0 0 -0.0827"/>
+            <geometry>
+                <mesh filename="package://soccer_description/meshes/soccerbot v4/Right Calve.dae" scale="1 1 1"/>
+            </geometry>
+            <material name="black" />
+        </visual>
+    </link>
+    <link name="right_ankle">
         <inertial>
             <mass value="153.186"/>
             <origin rpy="0 0 0" xyz="0  0  0"/>
-            <inertia ixx="0.205" ixy="0.0" ixz="0" iyy="0.173" iyz="0.038" izz="0.060"/>
-        </inertial>
-        <collision name="collision">
-            <origin rpy="0 1.5708 0" xyz="0 0.01031 -0.02014"/>
-            <geometry>
-                <box size="0.090769 0.0506 0.042"/>
-            </geometry>
-        </collision>
-        <visual name="visual">
-            <origin rpy="0  0  0" xyz="0  0  0"/>
-            <geometry>
-                <mesh filename="package://soccer_description/meshes/soccerbot v4/Left Ankle.stl" scale="0.001 0.001 0.001"/>
-            </geometry>
-            <material name="black" />
-        </visual>
-    </link>
-    <link name="left_calve">
-        <inertial>
-            <mass value="86.598"/>
-            <origin rpy="0  0  0" xyz="0 0  0"/>
-            <inertia ixx="0.077" ixy="0" ixz="0" iyy="0.019" iyz="0.001" izz="0.085"/>
-        </inertial>
-        <collision name="collision">
-            <origin rpy="0  1.5708  0" xyz="0      -0.03385  0"/>
-            <geometry>
-                <box size="0.031883 0.105683 0.048"/>
-            </geometry>
-        </collision>
-        <visual name="visual">
-            <origin rpy="0  0  0" xyz="0 -0.0827  0"/>
-            <geometry>
-                <mesh filename="package://soccer_description/meshes/soccerbot v4/Left Calve.stl" scale="0.001 0.001 0.001"/>
-            </geometry>
-            <material name="black" />
-        </visual>
-    </link>
-    <link name="left_foot">
+            <inertia ixx="0.038" ixy="0" ixz="0" iyy="0.060" iyz="0.038" izz="0.173"/>
+        </inertial>
+        <collision name="collision">
+            <origin rpy="0 0 0" xyz="-0.02014 0 0.01031"/>
+            <geometry>
+                <box size="0.090769 0.042 0.0506"/>
+            </geometry>
+        </collision>
+        <visual name="visual">
+            <origin rpy="0  0  0" xyz="0  0  0"/>
+            <geometry>
+                <mesh filename="package://soccer_description/meshes/soccerbot v4/Right Ankle.dae" scale="1 1 1"/>
+            </geometry>
+            <material name="black" />
+        </visual>
+    </link>
+    <link name="right_foot">
         <inertial>
             <mass value="23.216"/>
             <origin rpy="0 0 0" xyz="0  0  0"/>
-            <inertia ixx="0.026" ixy="0" ixz="0" iyy="0.023" iyz="0" izz="0.013"/>
-        </inertial>
-        <collision name="collision">
-            <origin rpy="0 1.5708 0" xyz="-0.00401 -0.00737  0.00385"/>
-            <geometry>
-                <box size="0.09 0.03674 0.07"/>
+            <inertia ixx="0.013" ixy="0" ixz="0.001" iyy="0.025" iyz="0.002" izz="0.022"/>
+        </inertial>
+        <collision name="collision">
+            <origin rpy="0 0 0" xyz="0.00385 -0.00401 -0.00737"/>
+            <geometry>
+                <box size="0.09 0.07 0.03674"/>
             </geometry>
             <contact_coefficients mu ="100.0" />
@@ -112,5 +192,25 @@
             <origin rpy="0  0  0" xyz="0  0  0"/>
             <geometry>
-                <mesh filename="package://soccer_description/meshes/soccerbot v4/Left Foot.stl" scale="0.001 0.001 0.001"/>
+                <mesh filename="package://soccer_description/meshes/soccerbot v4/Right Foot.dae" scale="1 1 1"/>
+            </geometry>
+            <material name="black" />
+        </visual>
+    </link>
+    <link name="left_hip_side">
+        <inertial>
+            <mass value="9.364"/>
+            <origin rpy="0  0  0" xyz="0  0  0"/>
+            <inertia ixx="0.004" ixy="0" ixz="0" iyy="0.007" iyz="0" izz="0.004"/>
+        </inertial>
+        <collision name="collision">
+            <origin rpy="0  0  0" xyz="0 0 0.00899"/>
+            <geometry>
+                <box size="0.0485 0.022 0.0039"/>
+            </geometry>
+        </collision>
+        <visual name="visual">
+            <origin rpy="0  0  0" xyz="0  0  0"/>
+            <geometry>
+                <mesh filename="package://soccer_description/meshes/soccerbot v4/Left Hip Side.dae" scale="1 1 1"/>
             </geometry>
             <material name="black" />
@@ -119,38 +219,18 @@
     <link name="left_hip_front">
         <inertial>
-            <mass value="153.238"/>
-            <origin rpy="0  0  0" xyz="0  0  0"/>
-            <inertia ixx="0.205" ixy="0" ixz="0" iyy="0.173" iyz="0.038" izz="0.060"/>
-        </inertial>
-        <collision name="collision">
-            <origin rpy="0 1.5707 0" xyz="0 -0.01332 -0.02187"/> <!-- 0.01332-->
-            <geometry>
-                <box size="0.083747 0.0506 0.04885"/>
-            </geometry>
-        </collision>
-        <visual name="visual">
-            <origin rpy="0  0  0" xyz="0  0  0"/>
-            <geometry>
-                <mesh filename="package://soccer_description/meshes/soccerbot v4/Left Hip Front.stl" scale="0.001 0.001 0.001"/>
-            </geometry>
-            <material name="black" />
-        </visual>
-    </link>
-    <link name="left_hip_side">
-        <inertial>
-            <mass value="9.364"/>
-            <origin rpy="0  0  0" xyz="0  0  0"/>
-            <inertia ixx="0.007" ixy="0" ixz="0" iyy="0.004" iyz="0" izz="0.004"/>
-        </inertial>
-        <collision name="collision">
-            <origin rpy="0  0  0" xyz="0       0.00899  0"/>
-            <geometry>
-                <box size="0.022 0.039 0.0475"/>
-            </geometry>
-        </collision>
-        <visual name="visual">
-            <origin rpy="0  0  0" xyz="0  0  0"/>
-            <geometry>
-                <mesh filename="package://soccer_description/meshes/soccerbot v4/Left Hip Side.stl" scale="0.001 0.001 0.001"/>
+            <mass value="153.186"/>
+            <origin rpy="0 0 0" xyz="0 0 0"/>
+            <inertia ixx="0.060" ixy="0.000" ixz="-0.038" iyy="0.205" iyz="0.000" izz="0.173"/>
+        </inertial>
+        <collision name="collision">
+            <origin rpy="0 0 0" xyz="-0.02187 0 -0.01332"/>
+            <geometry>
+                <box size="0.083747 0.04885 0.0506"/>
+            </geometry>
+        </collision>
+        <visual name="visual">
+            <origin rpy="0  0  0" xyz="0  0  0"/>
+            <geometry>
+                <mesh filename="package://soccer_description/meshes/soccerbot v4/Left Hip Front.dae" scale="1 1 1"/>
             </geometry>
             <material name="black" />
@@ -160,91 +240,71 @@
         <inertial>
             <mass value="21.438"/>
-            <origin rpy="0  0  0" xyz="0  0  0"/>
-            <inertia ixx="0.063" ixy="0" ixz="0" iyy="0.011" iyz="0" izz="0.072"/>
-        </inertial>
-        <collision name="collision">
-            <origin rpy="0 1.5708 0" xyz="0     -0.0445  0"/>
-            <geometry>
-                <box size="0.022 0.111 0.048"/>
-            </geometry>
-        </collision>
-        <visual name="visual">
-            <origin rpy="0  0  0" xyz="0  0  0"/>
-            <geometry>
-                <mesh filename="package://soccer_description/meshes/soccerbot v4/Left Thigh.stl" scale="0.001 0.001 0.001"/>
-            </geometry>
-            <material name="black" />
-        </visual>
-    </link>
-    <link name="neck">
-        <inertial>
-            <mass value="70.031"/>
-            <origin rpy="0  0  0" xyz="0  0  0"/>
-            <inertia ixx="0.009" ixy="0" ixz="0" iyy="0.031" iyz="0" izz="0.034"/>
-        </inertial>
-        <collision name="collision">
-            <origin rpy="0  0  0" xyz="0      0.0165  0"/>
-            <geometry>
-                <box size="0.0523 0.033 0.022"/>
-            </geometry>
-        </collision>
-        <visual name="visual">
-            <origin rpy="0  0  0" xyz="0  0  0"/>
-            <geometry>
-                <mesh filename="package://soccer_description/meshes/soccerbot v4/Neck.stl" scale="0.001 0.001 0.001"/>
-            </geometry>
-            <material name="black" />
-        </visual>
-    </link>
-    <link name="right_ankle">
-        <inertial>
-            <mass value="153.238"/>
             <origin rpy="0 0 0" xyz="0  0  0"/>
-            <inertia ixx="0.205" ixy="0" ixz="0" iyy="0.173" iyz="0.038" izz="0.060"/>
-        </inertial>
-        <collision name="collision">
-            <origin rpy="0 1.5708 0" xyz="0 0.01031 -0.02014"/>
-            <geometry>
-                <box size="0.090769 0.0506 0.042"/>
-            </geometry>
-        </collision>
-        <visual name="visual">
-            <origin rpy="0  0  0" xyz="0  0  0"/>
-            <geometry>
-                <mesh filename="package://soccer_description/meshes/soccerbot v4/Right Ankle.stl" scale="0.001 0.001 0.001"/>
-            </geometry>
-            <material name="black" />
-        </visual>
-    </link>
-    <link name="right_calve">
-        <inertial>
-            <mass value="86.598"/>
+            <inertia ixx="0.063" ixy="0" ixz="0.002" iyy="0.063" iyz="0" izz="0.011"/>
+        </inertial>
+        <collision name="collision">
+            <origin rpy="0 0 0" xyz="0 0 -0.0445"/>
+            <geometry>
+                <box size="0.022 0.048 0.111"/>
+            </geometry>
+        </collision>
+        <visual name="visual">
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
Commit message: Updated IMU readings

File: models/soccerbot/model.xacro (robot description, xacro)
@@ -35,5 +35,5 @@
     </link>
     <link name="camera" />
-    <link name="imu" />
+    <link name="imu_link" />
     <link name="neck">
         <inertial>
@@ -63,5 +63,5 @@
         </inertial>
         <collision name="collision">
-            <origin rpy="0  0  0" xyz="0 0 0.01995"/>
+            <origin rpy="0  0  0" xyz="0.0122 0 0.01995"/>
             <geometry>
                 <box size="0.0712 0.094 0.0839"/>
@@ -407,9 +407,7 @@
     <joint name="torso_imu" type="fixed">
         <parent link="torso"/>
-        <child link="imu"/>
-        <origin rpy="0 0 0" xyz="-0.03095 -0.0562  0.001286"/>
-        <axis xyz="0 0  0"/>
-        <dynamics damping="0.0" friction="2000.0" />
-        <limit effort="0" lower="0" upper="0" velocity="0"/>
+        <child link="imu_link"/>
+        <origin rpy="0 0 0" xyz="0.1 0 0.0075"/>
+        <axis xyz="0 0 0"/>
     </joint>
     <joint name="torso_right_hip_side" type="revolute">
@@ -441,7 +439,7 @@
         <child link="right_calve"/>
         <origin rpy="0 0 0" xyz="0 0 -0.0929"/>
-        <axis xyz="0 1 0"/>
-        <dynamics damping="0.0" friction="2000.0" />
-        <limit effort="31000.0" lower="0" upper="2.793" velocity="1.0"/>
+        <axis xyz="0 -1 0"/>
+        <dynamics damping="0.0" friction="2000.0" />
+        <limit effort="31000.0" lower="-2.793" upper="0" velocity="1.0"/>
     </joint>
     <joint name="right_calve_ankle" type="revolute">
@@ -489,7 +487,7 @@
         <child link="left_calve"/>
         <origin rpy="0 0 0" xyz="0 0 -0.09290"/>
-        <axis xyz="0 1 0"/>
-        <dynamics damping="0.0" friction="2000.0" />
-        <limit effort="31000.0" lower="0" upper="2.793" velocity="1.0"/>
+        <axis xyz="0 -1 0"/>
+        <dynamics damping="0.0" friction="2000.0" />
+        <limit effort="31000.0" lower="-2.793" upper="0" velocity="1.0"/>
     </joint>
     <joint name="left_calve_ankle" type="revolute">

Commit message: Added frictions on arms

File: models/soccerbot/model.xacro (robot description, xacro)
@@ -63,5 +63,5 @@
         </inertial>
         <collision name="collision">
-            <origin rpy="0  0  0" xyz="0.0122 0 0.01995"/>
+            <origin rpy="0  0  0" xyz="0.01735 0 0.01995"/>
             <geometry>
                 <box size="0.0712 0.094 0.0839"/>
@@ -743,4 +743,4 @@
             <mechanicalReduction>1</mechanicalReduction>
         </actuator>
-    </transmission>
+    </transmission>/
 </robot>
