Commit message: This time i got the inertias correct

File: models/soccerbot/model.xacro (robot description, xacro)
@@ -18,6 +18,6 @@
         <inertial>
             <mass value="1529.201"/>
-            <origin rpy="0 0 0" xyz="0 0 0"/>
-            <inertia ixx="5.590" ixy="0.006" ixz="0.063" iyy="8.698" iyz="-0.056" izz="3.302"/>
+            <origin rpy="0 0 0" xyz="0.0082498 -0.0017440 -0.0522479"/>
+            <inertia ixx="4.323" ixy="0.006" ixz="0.040" iyy="5.198" iyz="-0.015" izz="3.567"/>
         </inertial>
         <collision name="collision">
@@ -39,6 +39,6 @@
         <inertial>
             <mass value="11.294"/>
-            <origin rpy="0  0  0" xyz="0  0  0"/>
-            <inertia ixx="0.006" ixy="0" ixz="0" iyy="0.002" iyz="0" izz="0.005"/>
+            <origin rpy="0  0  0" xyz="0 -0.0006476 0.0092453"/>
+            <inertia ixx="0.005" ixy="0" ixz="0" iyy="0.001" iyz="0" izz="0.005"/>
         </inertial>
         <collision name="collision">
@@ -59,6 +59,6 @@
         <inertial>
             <mass value="282.919"/>
-            <origin rpy="0  0  0" xyz="0  0  0"/>
-            <inertia ixx="0.392" ixy="-0.011" ixz="-0.229" iyy="0.550" iyz="-0.011" izz="0.320"/>
+            <origin rpy="0  0  0" xyz="0.0237166 0.0018096 0.0255966"/>
+            <inertia ixx="0.206" ixy="0.001" ixz="-0.057" iyy="0.206" iyz="0.003" izz="0.160"/>
         </inertial>
         <collision name="collision">
@@ -79,6 +79,6 @@
         <inertial>
             <mass value="9.364"/>
-            <origin rpy="0  0  0" xyz="0  0  0"/>
-            <inertia ixx="0.004" ixy="0" ixz="0" iyy="0.007" iyz="0" izz="0.004"/>
+            <origin rpy="0  0  0" xyz="0.0003695 0.0000 0.01689"/>
+            <inertia ixx="0.002" ixy="0.000" ixz="0.000" iyy="0.005" iyz="0.000" izz="0.004"/>
         </inertial>
         <collision name="collision">
@@ -99,6 +99,6 @@
         <inertial>
             <mass value="153.186"/>
-            <origin rpy="0 0 0" xyz="0 0 0"/>
-            <inertia ixx="0.060" ixy="0.000" ixz="-0.038" iyy="0.205" iyz="0.000" izz="0.173"/>
+            <origin rpy="0 0 0" xyz="-0.02093 0 -0.011313"/>
+            <inertia ixx="0.041" ixy="0.000" ixz="-0.002" iyy="0.118" iyz="0.000" izz="0.106"/>
         </inertial>
         <collision name="collision">
@@ -119,69 +119,190 @@
         <inertial>
             <mass value="21.438"/>
+            <origin rpy="0 0 0" xyz="0.0019422 0.0001419 -0.0469409"/>
+            <inertia ixx="0.025" ixy="0.002" ixz="0.000" iyy="0.016" iyz="0.000" izz="0.010"/>
+        </inertial>
+        <collision name="collision">
+            <origin rpy="0 0 0" xyz="0 0 -0.0445"/>
+            <geometry>
+                <box size="0.022 0.048 0.111"/>
+            </geometry>
+        </collision>
+        <visual name="visual">
+            <origin rpy="0  0  0" xyz="0  0  0"/>
+            <geometry>
+                <mesh filename="package://soccer_description/meshes/soccerbot v4/Right Thigh.dae" scale="1 1 1"/>
+            </geometry>
+            <material name="black" />
+        </visual>
+    </link>
+    <link name="right_calve">
+        <inertial>
+            <mass value="86.547"/>
+            <origin rpy="0  0  0" xyz="0 -0.0003259 -0.0150123"/>
+            <inertia ixx="0.054" ixy="0.000" ixz="0.000" iyy="0.046" iyz="0.001" izz="0.019"/>
+        </inertial>
+        <collision name="collision">
+            <origin rpy="0 0 0" xyz="0 0 -0.03385"/>
+            <geometry>
+                <box size="0.031883 0.048 0.105683"/>
+            </geometry>
+        </collision>
+        <visual name="visual">
+            <origin rpy="0 0 0" xyz="0 0 -0.0827"/>
+            <geometry>
+                <mesh filename="package://soccer_description/meshes/soccerbot v4/Right Calve.dae" scale="1 1 1"/>
+            </geometry>
+            <material name="black" />
+        </visual>
+    </link>
+    <link name="right_ankle">
+        <inertial>
+            <mass value="153.186"/>
+            <origin rpy="0 0 0" xyz="-0.020939 0.000 0.011313"/>
+            <inertia ixx="0.041" ixy="0.000" ixz="0.002" iyy="0.118" iyz="0.000" izz="0.106"/>
+        </inertial>
+        <collision name="collision">
+            <origin rpy="0 0 0" xyz="-0.02014 0 0.01031"/>
+            <geometry>
+                <box size="0.090769 0.042 0.0506"/>
+            </geometry>
+        </collision>
+        <visual name="visual">
+            <origin rpy="0  0  0" xyz="0  0  0"/>
+            <geometry>
+                <mesh filename="package://soccer_description/meshes/soccerbot v4/Right Ankle.dae" scale="1 1 1"/>
+            </geometry>
+            <material name="black" />
+        </visual>
+    </link>
+    <link name="right_foot">
+        <inertial>
+            <mass value="23.216"/>
+            <origin rpy="0 0 0" xyz="-0.020939 0.0 0.011313"/>
+            <inertia ixx="0.006" ixy="0.000" ixz="0.000" iyy="0.018" iyz="0.000" izz="0.022"/>
+        </inertial>
+        <collision name="collision">
+            <origin rpy="0 0 0" xyz="0.00385 -0.00401 -0.00737"/>
+            <geometry>
+                <box size="0.09 0.07 0.03674"/>
+            </geometry>
+            <contact_coefficients mu ="100.0" />
+        </collision>
+        <visual name="visual">
+            <origin rpy="0  0  0" xyz="0  0  0"/>
+            <geometry>
+                <mesh filename="package://soccer_description/meshes/soccerbot v4/Right Foot.dae" scale="1 1 1"/>
+            </geometry>
+            <material name="black" />
+        </visual>
+    </link>
+    <link name="left_hip_side">
+        <inertial>
+            <mass value="9.364"/>
+            <origin rpy="0  0  0" xyz="0.0003695 0.0000 0.01689"/>
+            <inertia ixx="0.002" ixy="0.000" ixz="0.000" iyy="0.005" iyz="0.000" izz="0.004"/>
+        </inertial>
+        <collision name="collision">
+            <origin rpy="0  0  0" xyz="0 0 0.00899"/>
+            <geometry>
+                <box size="0.0485 0.022 0.0039"/>
+            </geometry>
+        </collision>
+        <visual name="visual">
+            <origin rpy="0  0  0" xyz="0  0  0"/>
+            <geometry>
+                <mesh filename="package://soccer_description/meshes/soccerbot v4/Left Hip Side.dae" scale="1 1 1"/>
+            </geometry>
+            <material name="black" />
+        </visual>
+    </link>
+    <link name="left_hip_front">
+        <inertial>
+            <mass value="153.186"/>
+            <origin rpy="0 0 0" xyz="-0.02093 0 -0.011313"/>
+            <inertia ixx="0.041" ixy="0.000" ixz="-0.002" iyy="0.118" iyz="0.000" izz="0.106"/>
+        </inertial>
+        <collision name="collision">
+            <origin rpy="0 0 0" xyz="-0.02187 0 -0.01332"/>
+            <geometry>
+                <box size="0.083747 0.04885 0.0506"/>
+            </geometry>
+        </collision>
+        <visual name="visual">
+            <origin rpy="0  0  0" xyz="0  0  0"/>
+            <geometry>
+                <mesh filename="package://soccer_description/meshes/soccerbot v4/Left Hip Front.dae" scale="1 1 1"/>
+            </geometry>
+            <material name="black" />
+        </visual>
+    </link>
+    <link name="left_thigh">
+        <inertial>
+            <mass value="21.438"/>
+            <origin rpy="0 0 0" xyz="0.0019422 -0.0001419 -0.0469409"/>
+            <inertia ixx="0.025" ixy="-0.002" ixz="0.000" iyy="0.016" iyz="0.000" izz="0.010"/>
+        </inertial>
+        <collision name="collision">
+            <origin rpy="0 0 0" xyz="0 0 -0.0445"/>
+            <geometry>
+                <box size="0.022 0.048 0.111"/>
+            </geometry>
+        </collision>
+        <visual name="visual">
+            <origin rpy="0  0  0" xyz="0  0  0"/>
+            <geometry>
+                <mesh filename="package://soccer_description/meshes/soccerbot v4/Left Thigh.dae" scale="1 1 1"/>
+            </geometry>
+            <material name="black" />
+        </visual>
+    </link>
+    <link name="left_calve">
+        <inertial>
+            <mass value="86.547"/>
+            <origin rpy="0  0  0" xyz="0 0.0003259 -0.0150123"/>
+            <inertia ixx="0.054" ixy="0.000" ixz="0.000" iyy="0.046" iyz="-0.001" izz="0.019"/>
+        </inertial>
+        <collision name="collision">
+            <origin rpy="0 0 0" xyz="0 0 -0.03385"/>
+            <geometry>
+                <box size="0.031883 0.048 0.105683"/>
+            </geometry>
+        </collision>
+        <visual name="visual">
+            <origin rpy="0 0 0" xyz="0 0 -0.0827"/>
+            <geometry>
+                <mesh filename="package://soccer_description/meshes/soccerbot v4/Left Calve.dae" scale="1 1 1"/>
+            </geometry>
+            <material name="black" />
+        </visual>
+    </link>
+    <link name="left_ankle">
+        <inertial>
+            <mass value="153.186"/>
+            <origin rpy="0 0 0" xyz="-0.020939 0.000 0.011313"/>
+            <inertia ixx="0.041" ixy="0.000" ixz="0.002" iyy="0.118" iyz="0.000" izz="0.106"/>
+        </inertial>
+        <collision name="collision">
+            <origin rpy="0 0 0" xyz="-0.02014 0 0.01031"/>
+            <geometry>
+                <box size="0.090769 0.042 0.0506"/>
+            </geometry>
+        </collision>
+        <visual name="visual">
             <origin rpy="0 0 0" xyz="0  0  0"/>
-            <inertia ixx="0.063" ixy="0" ixz="0.002" iyy="0.063" iyz="0" izz="0.011"/>
-        </inertial>
-        <collision name="collision">
-            <origin rpy="0 0 0" xyz="0 0 -0.0445"/>
-            <geometry>
-                <box size="0.022 0.048 0.111"/>
-            </geometry>
-        </collision>
-        <visual name="visual">
-            <origin rpy="0  0  0" xyz="0  0  0"/>
-            <geometry>
-                <mesh filename="package://soccer_description/meshes/soccerbot v4/Right Thigh.dae" scale="1 1 1"/>
-            </geometry>
-            <material name="black" />
-        </visual>
-    </link>
-    <link name="right_calve">
-        <inertial>
-            <mass value="86.547"/>
-            <origin rpy="0  0  0" xyz="0 0 0"/>
-            <inertia ixx="0.072" ixy="0" ixz="0" iyy="0.443" iyz="0.003" izz="0.019"/>
-        </inertial>
-        <collision name="collision">
-            <origin rpy="0 0 0" xyz="0 0 -0.03385"/>
-            <geometry>
-                <box size="0.031883 0.048 0.105683"/>
-            </geometry>
-        </collision>
-        <visual name="visual">
-            <origin rpy="0 0 0" xyz="0 0 -0.0827"/>
-            <geometry>
-                <mesh filename="package://soccer_description/meshes/soccerbot v4/Right Calve.dae" scale="1 1 1"/>
-            </geometry>
-            <material name="black" />
-        </visual>
-    </link>
-    <link name="right_ankle">
-        <inertial>
-            <mass value="153.186"/>
-            <origin rpy="0 0 0" xyz="0  0  0"/>
-            <inertia ixx="0.038" ixy="0" ixz="0" iyy="0.060" iyz="0.038" izz="0.173"/>
-        </inertial>
-        <collision name="collision">
-            <origin rpy="0 0 0" xyz="-0.02014 0 0.01031"/>
-            <geometry>
-                <box size="0.090769 0.042 0.0506"/>
-            </geometry>
-        </collision>
-        <visual name="visual">
-            <origin rpy="0  0  0" xyz="0  0  0"/>
-            <geometry>
-                <mesh filename="package://soccer_description/meshes/soccerbot v4/Right Ankle.dae" scale="1 1 1"/>
-            </geometry>
-            <material name="black" />
-        </visual>
-    </link>
-    <link name="right_foot">
+            <geometry>
+                <mesh filename="package://soccer_description/meshes/soccerbot v4/Left Ankle.dae" scale="1 1 1"/>
+            </geometry>
+            <material name="black" />
+        </visual>
+    </link>
+    <link name="left_foot">
         <inertial>
             <mass value="23.216"/>
-            <origin rpy="0 0 0" xyz="0  0  0"/>
-            <inertia ixx="0.013" ixy="0" ixz="0.001" iyy="0.025" iyz="0.002" izz="0.022"/>
-        </inertial>
-        <collision name="collision">
-            <origin rpy="0 0 0" xyz="0.00385 -0.00401 -0.00737"/>
+            <origin rpy="0 0 0" xyz="-0.020939 0.0 0.011313"/>
+            <inertia ixx="0.006" ixy="0.000" ixz="0.000" iyy="0.018" iyz="0.000" izz="0.022"/>
+        </inertial>
+        <collision name="collision">
+            <origin rpy="0 0 0" xyz="0.00385 0.00401 -0.00737 "/>
             <geometry>
                 <box size="0.09 0.07 0.03674"/>
@@ -192,125 +313,4 @@
             <origin rpy="0  0  0" xyz="0  0  0"/>
             <geometry>
-                <mesh filename="package://soccer_description/meshes/soccerbot v4/Right Foot.dae" scale="1 1 1"/>
-            </geometry>
-            <material name="black" />
-        </visual>
-    </link>
-    <link name="left_hip_side">
-        <inertial>
-            <mass value="9.364"/>
-            <origin rpy="0  0  0" xyz="0  0  0"/>
-            <inertia ixx="0.004" ixy="0" ixz="0" iyy="0.007" iyz="0" izz="0.004"/>
-        </inertial>
-        <collision name="collision">
-            <origin rpy="0  0  0" xyz="0 0 0.00899"/>
-            <geometry>
-                <box size="0.0485 0.022 0.0039"/>
-            </geometry>
-        </collision>
-        <visual name="visual">
-            <origin rpy="0  0  0" xyz="0  0  0"/>
-            <geometry>
-                <mesh filename="package://soccer_description/meshes/soccerbot v4/Left Hip Side.dae" scale="1 1 1"/>
-            </geometry>
-            <material name="black" />
-        </visual>
-    </link>
-    <link name="left_hip_front">
-        <inertial>
-            <mass value="153.186"/>
-            <origin rpy="0 0 0" xyz="0 0 0"/>
-            <inertia ixx="0.060" ixy="0.000" ixz="-0.038" iyy="0.205" iyz="0.000" izz="0.173"/>
-        </inertial>
-        <collision name="collision">
-            <origin rpy="0 0 0" xyz="-0.02187 0 -0.01332"/>
-            <geometry>
-                <box size="0.083747 0.04885 0.0506"/>
-            </geometry>
-        </collision>
-        <visual name="visual">
-            <origin rpy="0  0  0" xyz="0  0  0"/>
-            <geometry>
-                <mesh filename="package://soccer_description/meshes/soccerbot v4/Left Hip Front.dae" scale="1 1 1"/>
-            </geometry>
-            <material name="black" />
-        </visual>
-    </link>
-    <link name="left_thigh">
-        <inertial>
-            <mass value="21.438"/>
-            <origin rpy="0 0 0" xyz="0  0  0"/>
-            <inertia ixx="0.063" ixy="0" ixz="0.002" iyy="0.063" iyz="0" izz="0.011"/>
-        </inertial>
-        <collision name="collision">
-            <origin rpy="0 0 0" xyz="0 0 -0.0445"/>
-            <geometry>
-                <box size="0.022 0.048 0.111"/>
-            </geometry>
-        </collision>
-        <visual name="visual">
-            <origin rpy="0  0  0" xyz="0  0  0"/>
-            <geometry>
-                <mesh filename="package://soccer_description/meshes/soccerbot v4/Left Thigh.dae" scale="1 1 1"/>
-            </geometry>
-            <material name="black" />
-        </visual>
-    </link>
-    <link name="left_calve">
-        <inertial>
-            <mass value="86.547"/>
-            <origin rpy="0  0  0" xyz="0 0 0"/>
-            <inertia ixx="0.072" ixy="0" ixz="0" iyy="0.443" iyz="-0.003" izz="0.019"/>
-        </inertial>
-        <collision name="collision">
-            <origin rpy="0 0 0" xyz="0 0 -0.03385"/>
-            <geometry>
-                <box size="0.031883 0.048 0.105683"/>
-            </geometry>
-        </collision>
-        <visual name="visual">
-            <origin rpy="0 0 0" xyz="0 0 -0.0827"/>
-            <geometry>
-                <mesh filename="package://soccer_description/meshes/soccerbot v4/Left Calve.dae" scale="1 1 1"/>
-            </geometry>
-            <material name="black" />
-        </visual>
-    </link>
-    <link name="left_ankle">
-        <inertial>
-            <mass value="153.186"/>
-            <origin rpy="0 0 0" xyz="0  0  0"/>
-            <inertia ixx="0.038" ixy="0" ixz="0" iyy="0.060" iyz="-0.038" izz="0.173"/>
-        </inertial>
-        <collision name="collision">
-            <origin rpy="0 0 0" xyz="-0.02014 0 0.01031"/>
-            <geometry>
-                <box size="0.090769 0.042 0.0506"/>
-            </geometry>
-        </collision>
-        <visual name="visual">
-            <origin rpy="0 0 0" xyz="0  0  0"/>
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
Commit message: Update model.xacro

File: models/soccerbot/model.xacro (robot description, xacro)
@@ -455,5 +455,5 @@
         <child link="right_foot"/>
         <origin rpy="0 0 0" xyz="0 0 0"/>
-        <axis xyz="1 0 0"/>
+        <axis xyz="-1 0 0"/>
         <dynamics damping="0.0" friction="2000.0" />
         <limit effort="31000.0" lower="-0.785" upper="0.785" velocity="1.0"/>
@@ -503,5 +503,5 @@
         <child link="left_foot"/>
         <origin rpy="0 0 0" xyz="0 0 0"/>
-        <axis xyz="-1 0 0"/>
+        <axis xyz="1 0 0"/>
         <dynamics damping="0.0" friction="2000.0" />
         <limit effort="31000.0" lower="-0.785" upper="0.785" velocity="1.0"/>

Commit message: Updated xacro

File: models/soccerbot/model.xacro (robot description, xacro)
@@ -5,12 +5,4 @@
     <!-- Import Rviz colors -->
     <xacro:include filename="$(find soccer_description)/models/soccerbot/materials.xacro" />
-    <!-- Joint to keep the robot up in midair -->
-    <!--   <link name="world" />
-      <joint name="world_base_link" type="fixed">
-        <parent link="world"/>
-        <child link="base_link"/>
-        <origin rpy="0  0 0" xyz="0 0 0"/>
-        <axis xyz="1  0  0"/>
-      </joint> -->
     <!-- Links -->
     <link name="base_link" />
@@ -743,4 +735,4 @@
             <mechanicalReduction>1</mechanicalReduction>
         </actuator>
-    </transmission>
+    </transmission>/
 </robot>

Commit message: Uodated description

File: models/soccerbot/model.xacro (robot description, xacro)
@@ -447,5 +447,5 @@
         <child link="right_foot"/>
         <origin rpy="0 0 0" xyz="0 0 0"/>
-        <axis xyz="-1 0 0"/>
+        <axis xyz="1 0 0"/>
         <dynamics damping="0.0" friction="2000.0" />
         <limit effort="31000.0" lower="-0.785" upper="0.785" velocity="1.0"/>
@@ -465,5 +465,5 @@
         <axis xyz="1 0 0"/>
         <dynamics damping="0.0" friction="2000.0" />
-        <limit effort="31000.0" lower="-0.785" upper="1.571" velocity="1.0"/>
+        <limit effort="31000.0" lower="-1.571" upper="0.785" velocity="1.0"/>
     </joint>
     <joint name="left_hip_front_thigh" type="revolute">

Commit message: Fixed macro

File: models/soccerbot/model.xacro (robot description, xacro)
@@ -415,5 +415,5 @@
         <child link="right_hip_front"/>
         <origin rpy="0 0 0" xyz="0 0 0"/>
-        <axis xyz="1 0 0"/>
+        <axis xyz="-1 0 0"/>
         <dynamics damping="0.0" friction="2000.0" />
         <limit effort="31000.0" lower="-0.785" upper="1.571" velocity="1.0"/>
@@ -447,5 +447,5 @@
         <child link="right_foot"/>
         <origin rpy="0 0 0" xyz="0 0 0"/>
-        <axis xyz="1 0 0"/>
+        <axis xyz="-1 0 0"/>
         <dynamics damping="0.0" friction="2000.0" />
         <limit effort="31000.0" lower="-0.785" upper="0.785" velocity="1.0"/>
@@ -463,5 +463,5 @@
         <child link="left_hip_front"/>
         <origin rpy="0 0 0" xyz="0 0 0"/>
-        <axis xyz="1 0 0"/>
+        <axis xyz="-1 0 0"/>
         <dynamics damping="0.0" friction="2000.0" />
         <limit effort="31000.0" lower="-1.571" upper="0.785" velocity="1.0"/>
@@ -495,5 +495,5 @@
         <child link="left_foot"/>
         <origin rpy="0 0 0" xyz="0 0 0"/>
-        <axis xyz="1 0 0"/>
+        <axis xyz="-1 0 0"/>
         <dynamics damping="0.0" friction="2000.0" />
         <limit effort="31000.0" lower="-0.785" upper="0.785" velocity="1.0"/>
