Commit message: Refactoring

File: models/soccerbot/model.xacro (robot description, xacro)
@@ -22,5 +22,5 @@
             <origin rpy="0 0 0" xyz="0 0 0"/>
             <geometry>
-                <mesh filename="package://soccer_description/meshes/soccerbot v4/Torso.dae" scale="1 1 1"/>
+                <mesh filename="package://soccer_description/meshes/Torso.dae" scale="1 1 1"/>
             </geometry>
         </visual>
@@ -43,5 +43,5 @@
             <origin rpy="0  0  0" xyz="0  0  0"/>
             <geometry>
-                <mesh filename="package://soccer_description/meshes/soccerbot v4/Neck.dae" scale="1 1 1"/>
+                <mesh filename="package://soccer_description/meshes/Neck.dae" scale="1 1 1"/>
             </geometry>
             <material name="black" />
@@ -63,5 +63,5 @@
             <origin rpy="0  0  0" xyz="0  0  0"/>
             <geometry>
-                <mesh filename="package://soccer_description/meshes/soccerbot v4/Head.dae" scale="1 1 1"/>
+                <mesh filename="package://soccer_description/meshes/Head.dae" scale="1 1 1"/>
             </geometry>
             <material name="black" />
@@ -83,5 +83,5 @@
             <origin rpy="0  0  0" xyz="0  0  0"/>
             <geometry>
-                <mesh filename="package://soccer_description/meshes/soccerbot v4/Right Hip Side.dae" scale="1 1 1"/>
+                <mesh filename="package://soccer_description/meshes/Right Hip Side.dae" scale="1 1 1"/>
             </geometry>
             <material name="black" />
@@ -103,5 +103,5 @@
             <origin rpy="0  0  0" xyz="0  0  0"/>
             <geometry>
-                <mesh filename="package://soccer_description/meshes/soccerbot v4/Right Hip Front.dae" scale="1 1 1"/>
+                <mesh filename="package://soccer_description/meshes/Right Hip Front.dae" scale="1 1 1"/>
             </geometry>
             <material name="black" />
@@ -123,5 +123,5 @@
             <origin rpy="0  0  0" xyz="0  0  0"/>
             <geometry>
-                <mesh filename="package://soccer_description/meshes/soccerbot v4/Right Thigh.dae" scale="1 1 1"/>
+                <mesh filename="package://soccer_description/meshes/Right Thigh.dae" scale="1 1 1"/>
             </geometry>
             <material name="black" />
@@ -143,5 +143,5 @@
             <origin rpy="0 0 0" xyz="0 0 -0.0827"/>
             <geometry>
-                <mesh filename="package://soccer_description/meshes/soccerbot v4/Right Calve.dae" scale="1 1 1"/>
+                <mesh filename="package://soccer_description/meshes/Right Calve.dae" scale="1 1 1"/>
             </geometry>
             <material name="black" />
@@ -163,5 +163,5 @@
             <origin rpy="0  0  0" xyz="0  0  0"/>
             <geometry>
-                <mesh filename="package://soccer_description/meshes/soccerbot v4/Right Ankle.dae" scale="1 1 1"/>
+                <mesh filename="package://soccer_description/meshes/Right Ankle.dae" scale="1 1 1"/>
             </geometry>
             <material name="black" />
@@ -184,5 +184,5 @@
             <origin rpy="0  0  0" xyz="0  0  0"/>
             <geometry>
-                <mesh filename="package://soccer_description/meshes/soccerbot v4/Right Foot.dae" scale="1 1 1"/>
+                <mesh filename="package://soccer_description/meshes/Right Foot.dae" scale="1 1 1"/>
             </geometry>
             <material name="black" />
@@ -204,5 +204,5 @@
             <origin rpy="0  0  0" xyz="0  0  0"/>
             <geometry>
-                <mesh filename="package://soccer_description/meshes/soccerbot v4/Left Hip Side.dae" scale="1 1 1"/>
+                <mesh filename="package://soccer_description/meshes/Left Hip Side.dae" scale="1 1 1"/>
             </geometry>
             <material name="black" />
@@ -224,5 +224,5 @@
             <origin rpy="0  0  0" xyz="0  0  0"/>
             <geometry>
-                <mesh filename="package://soccer_description/meshes/soccerbot v4/Left Hip Front.dae" scale="1 1 1"/>
+                <mesh filename="package://soccer_description/meshes/Left Hip Front.dae" scale="1 1 1"/>
             </geometry>
             <material name="black" />
@@ -244,5 +244,5 @@
             <origin rpy="0  0  0" xyz="0  0  0"/>
             <geometry>
-                <mesh filename="package://soccer_description/meshes/soccerbot v4/Left Thigh.dae" scale="1 1 1"/>
+                <mesh filename="package://soccer_description/meshes/Left Thigh.dae" scale="1 1 1"/>
             </geometry>
             <material name="black" />
@@ -264,5 +264,5 @@
             <origin rpy="0 0 0" xyz="0 0 -0.0827"/>
             <geometry>
-                <mesh filename="package://soccer_description/meshes/soccerbot v4/Left Calve.dae" scale="1 1 1"/>
+                <mesh filename="package://soccer_description/meshes/Left Calve.dae" scale="1 1 1"/>
             </geometry>
             <material name="black" />
@@ -284,5 +284,5 @@
             <origin rpy="0 0 0" xyz="0  0  0"/>
             <geometry>
-                <mesh filename="package://soccer_description/meshes/soccerbot v4/Left Ankle.dae" scale="1 1 1"/>
+                <mesh filename="package://soccer_description/meshes/Left Ankle.dae" scale="1 1 1"/>
             </geometry>
             <material name="black" />
@@ -305,5 +305,5 @@
             <origin rpy="0  0  0" xyz="0  0  0"/>
             <geometry>
-                <mesh filename="package://soccer_description/meshes/soccerbot v4/Left Foot.dae" scale="1 1 1"/>
+                <mesh filename="package://soccer_description/meshes/Left Foot.dae" scale="1 1 1"/>
             </geometry>
             <material name="black" />
@@ -325,5 +325,5 @@
             <origin rpy="0  0  0" xyz="0  0  0"/>
             <geometry>
-                <mesh filename="package://soccer_description/meshes/soccerbot v4/Right Bicep.dae" scale="1 1 1"/>
+                <mesh filename="package://soccer_description/meshes/Right Bicep.dae" scale="1 1 1"/>
             </geometry>
             <material name="black" />
@@ -345,5 +345,5 @@
             <origin rpy="0  0  0" xyz="0  0  0"/>
             <geometry>
-                <mesh filename="package://soccer_description/meshes/soccerbot v4/Right Forearm.dae" scale="1 1 1"/>
+                <mesh filename="package://soccer_description/meshes/Right Forearm.dae" scale="1 1 1"/>
             </geometry>
             <material name="black" />
@@ -365,5 +365,5 @@
             <origin rpy="0  0  0" xyz="0  0  0"/>
             <geometry>
-                <mesh filename="package://soccer_description/meshes/soccerbot v4/Left Bicep.dae" scale="1 1 1"/>
+                <mesh filename="package://soccer_description/meshes/Left Bicep.dae" scale="1 1 1"/>
             </geometry>
             <material name="black" />
@@ -385,5 +385,5 @@
             <origin rpy="0  0  0" xyz="0  0  0"/>
             <geometry>
-                <mesh filename="package://soccer_description/meshes/soccerbot v4/Left Forearm.dae" scale="1 1 1"/>
+                <mesh filename="package://soccer_description/meshes/Left Forearm.dae" scale="1 1 1"/>
             </geometry>
             <material name="black" />
